Commit message: tweeks to ackermann vehicles

File: ackermann_vehicle_description/urdf/ackermann_1.xacro (robot description, xacro)
@@ -28,19 +28,19 @@
 -->
 <robot name="em_3905" xmlns:xacro="http://www.ros.org/wiki/xacro">
-	<macro name="cylinder_inertia" params="m r h">
+	<xacro:macro name="cylinder_inertia" params="m r h">
 		<inertia  ixx="${m*(3*r*r+h*h)/12}" ixy = "0" ixz = "0"
 		          iyy="${m*(3*r*r+h*h)/12}" iyz = "0"
 		          izz="${m*r*r/2}" />
-	</macro>
-	<macro name="box_inertia" params="m x y z">
+	</xacro:macro>
+	<xacro:macro name="box_inertia" params="m x y z">
 		<inertia  ixx="${m*(y*y+z*z)/12}" ixy = "0" ixz = "0"
 		          iyy="${m*(x*x+z*z)/12}" iyz = "0"
 		          izz="${m*(x*x+z*z)/12}" />
-	</macro>
-	<macro name="sphere_inertia" params="m r">
+	</xacro:macro>
+	<xacro:macro name="sphere_inertia" params="m r">
 		<inertia  ixx="${2*m*r*r/5}" ixy = "0" ixz = "0"
 		          iyy="${2*m*r*r/5}" iyz = "0"
 		          izz="${2*m*r*r/5}" />
-	</macro>
+	</xacro:macro>
   <!-- Degree-to-radian conversions -->
   <xacro:property name="degrees_45" value="0.785398163"/>

File: ackermann_vehicle_description/urdf/ackermann_2.xacro (robot description, xacro)
@@ -28,19 +28,19 @@
 -->
 <robot name="em_3905" xmlns:xacro="http://www.ros.org/wiki/xacro">
-	<macro name="cylinder_inertia" params="m r h">
+	<xacro:macro name="cylinder_inertia" params="m r h">
 		<inertia  ixx="${m*(3*r*r+h*h)/12}" ixy = "0" ixz = "0"
 		          iyy="${m*(3*r*r+h*h)/12}" iyz = "0"
 		          izz="${m*r*r/2}" />
-	</macro>
-	<macro name="box_inertia" params="m x y z">
+	</xacro:macro>
+	<xacro:macro name="box_inertia" params="m x y z">
 		<inertia  ixx="${m*(y*y+z*z)/12}" ixy = "0" ixz = "0"
 		          iyy="${m*(x*x+z*z)/12}" iyz = "0"
 		          izz="${m*(x*x+z*z)/12}" />
-	</macro>
-	<macro name="sphere_inertia" params="m r">
+	</xacro:macro>
+	<xacro:macro name="sphere_inertia" params="m r">
 		<inertia  ixx="${2*m*r*r/5}" ixy = "0" ixz = "0"
 		          iyy="${2*m*r*r/5}" iyz = "0"
 		          izz="${2*m*r*r/5}" />
-	</macro>
+	</xacro:macro>
   <!-- Degree-to-radian conversions -->
   <xacro:property name="degrees_45" value="0.785398163"/>
@@ -439,5 +439,5 @@
  </gazebo>
   <xacro:include filename="$(find velodyne_description)/urdf/VLP-16.urdf.xacro"/>
-  <VLP-16 parent="mount" name="velodyne" topic="/velodyne_points" hz="10" samples="440">
+  <VLP-16 parent="mount" name="velodyne" topic="/velodyne_points">
     <origin xyz="0 0 0.025" rpy="0 0 0" />
   </VLP-16>

Commit message: Enlarged ground plane image to proper scale for Gazebo sim.

File: ackermann_vehicle_description/urdf/ackermann_1.xacro (robot description, xacro)
@@ -48,5 +48,5 @@
   <!-- chassis_length is measured along the x axis, chassis_width
        along the y axis, and chassis_height along the z axis. -->
-  <xacro:property name="chassis_length" value="2.0"/><!-- 0.258 -->
+  <xacro:property name="chassis_length" value="2.61"/><!-- 0.258 -->
   <xacro:property name="chassis_width" value="0.8"/><!-- 0.168 -->
   <xacro:property name="chassis_height" value="0.3"/><!-- 0.1 -->
@@ -382,5 +382,5 @@
 	<!-- we can replace the z value with ${wheelRadius+chassisHeight+0.5}   							-->
   <joint name="camera_joint" type="fixed">
-    <origin xyz="${chassis_length/2} 0 ${(tire_dia/2)+chassis_height+.8}" rpy="0 1.0 0"/>
+    <origin xyz="${chassis_length/2} 0 ${(tire_dia/2)+chassis_height+.5}" rpy="0 .6 0"/>
     <parent link="chassis"/>
     <child link="camera"/>

Commit message: tweeks to urdf model

File: ackermann_vehicle_description/urdf/ackermann_1.xacro (robot description, xacro)
@@ -106,6 +106,6 @@
        6 V. servo_stall_torque is measured in N m. servo_no_load_speed is
        measured in rad/s. -->
-  <xacro:property name="servo_stall_torque" value="100"/><!--0.5649-->
-  <xacro:property name="servo_no_load_speed" value="20"/><!--4.553-->
+  <xacro:property name="servo_stall_torque" value="150"/><!-- Effort 0.5649-->
+  <xacro:property name="servo_no_load_speed" value="1"/><!--velocity 4.553-->
 	<xacro:property name="cameraSize" value=".05"/>
   <material name="battery_mat">
@@ -382,5 +382,5 @@
 	<!-- we can replace the z value with ${wheelRadius+chassisHeight+0.5}   							-->
   <joint name="camera_joint" type="fixed">
-    <origin xyz="${chassis_length/2} 0 ${(tire_dia/2)+chassis_height+.5}" rpy="0 .6 0"/>
+    <origin xyz="${(chassis_length/2)-1} 0 ${(tire_dia/2)+chassis_height+1.5}" rpy="0 .9 0"/> <!-- 0 .6 0 -->
     <parent link="chassis"/>
     <child link="camera"/>
